Commit message: add stairs terrain

File: urdf/atom01.urdf (robot description, URDF)
Before this commit: robot atom01urdf, 24 links, 23 joints
Links:
- link left_knee_link: geometry collision box size=0.08 0.10 0.24; visual mesh filename=../meshes/left_knee_link.STL
- link left_thigh_pitch_link: geometry collision box size=0.08 0.10 0.22; visual mesh filename=../meshes/left_thigh_pitch_link.STL
- link right_knee_link: geometry collision box size=0.08 0.10 0.24; visual mesh filename=../meshes/right_knee_link.STL
- link right_thigh_pitch_link: geometry collision box size=0.08 0.10 0.22; visual mesh filename=../meshes/right_thigh_pitch_link.STL
- link torso_link: geometry collision box size=0.16 0.16 0.22; visual mesh filename=../meshes/torso_link.STL
Joints:
- joint left_thigh_pitch_joint: limit lower=-1.57 upper=1.57 effort=120 velocity=25.0 -> lower=-2.094 upper=0.7854 effort=120 velocity=25.0
- joint right_thigh_pitch_joint: limit lower=-1.57 upper=1.57 effort=120 velocity=25.0 -> lower=-2.094 upper=0.7854 effort=120 velocity=25.0
